Commit message: Restore prototype Leader physical bounds and align collection limits with calibration

File: ros2_ws/src/xlerobot_description/urdf/leader_attachment.urdf.xacro (robot description, xacro)
@@ -7,4 +7,8 @@
   <xacro:property name="calibration" value="${xacro.load_yaml('$(arg calibration_file)')}"/>
   <xacro:property name="right" value="${calibration['joints']}"/>
+  <!-- The external Leader uses the frozen prototype's measured raw motor range.
+       Its copied Follower planning limits are not its physical attachment range.
+       Derive both URDF and hardware command limits identically; the Follower
+       retains its own calibrated limits and local teleop admission checks. -->
   <link name="leader_base"/>
   <xacro:macro name="leader_joint" params="name parent child calibration">
@@ -13,5 +17,5 @@
       <parent link="${parent}"/><child link="${child}"/>
       <origin xyz="0 0 0.05" rpy="0 0 0"/><axis xyz="0 0 1"/>
-      <limit lower="${calibration['limit_min']}" upper="${calibration['limit_max']}" velocity="3" effort="35"/>
+      <limit lower="${min(calibration['direction'] * (calibration['raw_min'] - calibration['offset']), calibration['direction'] * (calibration['raw_max'] - calibration['offset'])) * 2 * pi / 4096}" upper="${max(calibration['direction'] * (calibration['raw_min'] - calibration['offset']), calibration['direction'] * (calibration['raw_max'] - calibration['offset'])) * 2 * pi / 4096}" velocity="3" effort="35"/>
     </joint>
   </xacro:macro>
@@ -38,5 +42,5 @@
       <joint name="${name}">
         <command_interface name="position">
-          <param name="min">${calibration['limit_min']}</param><param name="max">${calibration['limit_max']}</param>
+          <param name="min">${min(calibration['direction'] * (calibration['raw_min'] - calibration['offset']), calibration['direction'] * (calibration['raw_max'] - calibration['offset'])) * 2 * pi / 4096}</param><param name="max">${max(calibration['direction'] * (calibration['raw_min'] - calibration['offset']), calibration['direction'] * (calibration['raw_max'] - calibration['offset'])) * 2 * pi / 4096}</param>
         </command_interface>
         <state_interface name="position"><param name="initial_value">${initial_value}</param></state_interface>
@@ -47,6 +51,6 @@
         <param name="raw_min">${calibration['raw_min']}</param>
         <param name="raw_max">${calibration['raw_max']}</param>
-        <param name="limit_min">${calibration['limit_min']}</param>
-        <param name="limit_max">${calibration['limit_max']}</param>
+        <param name="limit_min">${min(calibration['direction'] * (calibration['raw_min'] - calibration['offset']), calibration['direction'] * (calibration['raw_max'] - calibration['offset'])) * 2 * pi / 4096}</param>
+        <param name="limit_max">${max(calibration['direction'] * (calibration['raw_min'] - calibration['offset']), calibration['direction'] * (calibration['raw_max'] - calibration['offset'])) * 2 * pi / 4096}</param>
       </joint>
     </xacro:macro>
